File: infozilla/infozilla.kicad_sch (KiCad schematic)
At the start: 28 parts, among them J1 JST_S4B-XH-A-1, U1 Teensy4.1, U2 BMP280, U3 LIS3MDLTR, U4 LSM6DSOXTR, U5 MCP9808T-E_MS, U6 Adafruit_Ult_GPS, U7 Adafruit_RFM9x

Commit message: Added backup radio and debug LEDs
Parts:
- added C6, C7: 10uF, Capacitor_SMD:C_0805_2012Metric, symbol Device:C
- added C8: 0.1uF, Capacitor_SMD:C_0805_2012Metric, symbol Device:C
- added C9: 47pF, Capacitor_SMD:C_0805_2012Metric, symbol Device:C
- added D1: LED0, LED_SMD:LED_0603_1608Metric, symbol Device:LED
- added D2: LED1, LED_SMD:LED_0603_1608Metric, symbol Device:LED
- added D3: LED2, LED_SMD:LED_0603_1608Metric, symbol Device:LED
- added FB1, FB2: 120, Inductor_SMD:L_0402_1005Metric, symbol Device:FerriteBead
- added J2: Conn_01x05_Pin, Connector_PinHeader_2.54mm:PinHeader_1x05_P2.54mm_Vertical, symbol Connector:Conn_01x05_Pin
- added R6, R7, R8: 10k, Resistor_SMD:R_0805_2012Metric, symbol Device:R
Connections:
- net GND: now also C6.2, C7.2, C8.2, C9.2, D1.1 (K), D2.1 (K), D3.1 (K), FB2.1, FB2.2, J2.1 (Pin_1)
- net VDD: now also C6.1, FB1.1
- net RADIO2_TX: now reaches U1.26 (34_RX8)
- net RADIO2_TX: now also J2.2 (Pin_2)
- net RADIO2_RX: now reaches U1.27 (35_TX8)
- net RADIO2_RX: now also J2.3 (Pin_3)
- net RADIO2_RST: now reaches U1.28 (36_CS)
- net RADIO2_RST: now also J2.4 (Pin_4)
- net LED0: now reaches U1.4 (2_OUT2)
- net LED0: now also R6.1
- net LED1: now reaches U1.5 (3_LRCLK2)
- net LED1: now also R7.1
- net LED2: now reaches U1.6 (4_BCLK2)
- net LED2: now also R8.1
- new net: C7.1, C8.1, C9.1, FB1.2, J2.5 (Pin_5)
- new net: D3.2 (A), R8.2
- new net: D2.2 (A), R7.2
- new net: D1.2 (A), R6.2
- no-connect marks 59 -> 53
Other:
- note added: "Backup Radio"
- note added: "Debug LEDs"
