File: infozilla/infozilla.kicad_pcb (KiCad board)
At the start: 2 copper layers, 134 x 45 mm, 30 parts, among them J1 JST_S4B-XH-A-1, U1 Teensy4.1, U2 BMP280, U3 LIS3MDLTR, U4 LSM6DSOXTR, U5 MCP9808T-E_MS, U6 Adafruit_Ult_GPS, U7 Adafruit_RFM9x

Commit message: Added backup radio and debug LEDs
Parts:
- added C6: 10uF, Capacitor_SMD:C_0805_2012Metric, F.Cu at (214.0, 56.6)
- added C7: 10uF, Capacitor_SMD:C_0805_2012Metric, F.Cu at (215.0, 63.3)
- added C8: 0.1uF, Capacitor_SMD:C_0805_2012Metric, F.Cu at (214.5, 67.6)
- added C9: 47pF, Capacitor_SMD:C_0805_2012Metric, F.Cu at (217.9, 67.6)
- added D1: LED, LED_SMD:LED_0603_1608Metric, F.Cu at (110.6, 80.3)
- added D2: LED, LED_SMD:LED_0603_1608Metric, F.Cu at (113.3, 80.2)
- added D3: LED, LED_SMD:LED_0603_1608Metric, F.Cu at (116.5, 80.3)
- added FB1: FerriteBead, Inductor_SMD:L_0402_1005Metric, F.Cu at (213.0, 60.1)
- added FB2: FerriteBead, Inductor_SMD:L_0402_1005Metric, F.Cu at (215.9, 59.8)
- added J2: Conn_01x05_Pin, Connector_PinHeader_2.54mm:PinHeader_1x05_P2.54mm_Vertical, F.Cu at (222.2, 57.5)
- added R6: 10k, Resistor_SMD:R_0805_2012Metric, F.Cu at (111.1, 76.6)
- added R7: 10k, Resistor_SMD:R_0805_2012Metric, F.Cu at (113.6, 77.0)
- added R8: 10k, Resistor_SMD:R_0805_2012Metric, F.Cu at (116.8, 76.9)
- U5: value MCP9808T-E_MS -> MCP9808
Connections:
- U1 pad 26: unconnected-(U1-34_RX8-Pad26) -> /RADIO2_TX
- U1 pad 27: unconnected-(U1-35_TX8-Pad27) -> /RADIO2_RX
- U1 pad 28: unconnected-(U1-36_CS-Pad28) -> /RADIO2_RST
- U1 pad 4: unconnected-(U1-2_OUT2-Pad4) -> /LED0
- U1 pad 5: unconnected-(U1-3_LRCLK2-Pad5) -> /LED1
- U1 pad 6: unconnected-(U1-4_BCLK2-Pad6) -> /LED2
Routing:
- net /RADIO2_RX: track 0.00 -> 99.9 mm
- net /RADIO2_RST: track 0.00 -> 93.4 mm, vias 0 -> 1
- net /RADIO2_TX: track 0.00 -> 93.1 mm
- net VDD: track 35.5 -> 79.1 mm, vias 7 -> 12
- net GND: track 40.3 -> 77.3 mm, vias 12 -> 13
- net Net-(J2-Pin_5): track 0.00 -> 18.2 mm
- net /LED2: track 0.00 -> 13.4 mm, vias 0 -> 2
- net /LED0: track 0.00 -> 12.3 mm, vias 0 -> 2
- net /LED1: track 0.00 -> 11.7 mm, vias 0 -> 2
- net /RADIO_G2: track 137.4 -> 134.8 mm
- net /RADIO_G1: track 141.7 -> 139.1 mm
- net Net-(D1-A): track 0.00 -> 2.18 mm
- net Net-(D3-A): track 0.00 -> 1.92 mm
- net Net-(D2-A): track 0.00 -> 1.69 mm
- net /RADIO_G3: track 132.2 -> 130.6 mm
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Other:
- board text added: "RYLR998"

Commit message: Cutoff for LC2025
Parts:
- added G***: LOGO, custom_library:infozilla_vector, F.Cu at (161.2, 77.4)
- added G***: LOGO, custom_library:rocket_avionics_logo, F.Cu at (203.7, 77.4)
Other:
- board text added: "Ad astra per aspera."
