File: phoenix/mcu.kicad_sch (KiCad schematic)
At the start: 0 parts

Commit message: Finished schematics and almost done layouts of LC26 PCBs
Parts:
- added BZ1: Buzzer, Buzzer_Beeper:MagneticBuzzer_PUI_AT-0927-TT-6-R, symbol Device:Buzzer
- added D1: LED0, LED_SMD:LED_0603_1608Metric, symbol Device:LED
- added D2: LED1, LED_SMD:LED_0603_1608Metric, symbol Device:LED
- added D3: LED2, LED_SMD:LED_0603_1608Metric, symbol Device:LED
- added R1, R2: 4k7, Resistor_SMD:R_0603_1608Metric_Pad0.98x0.95mm_HandSolder, symbol Device:R
- added R3, R4, R5: 10k, Resistor_SMD:R_0603_1608Metric_Pad0.98x0.95mm_HandSolder, symbol Device:R
- added U13: Teensy4.1, custom_library:Teensy41_simplified, symbol custom_library:Teensy4.1_simplified
Connections:
- new net: D1.2 (A), R3.2
- new net: D2.2 (A), R4.2
- new net: D3.2 (A), R5.2
- new net: BZ1.1 (+), U13.25 (33_MCLK2)
- new net +3V3: R1.1, R2.1
- new net +5V: U13.48 (VIN)
- new net 3V3_EN: U13.27 (35_TX8)
- new net APOGEE_FIRE: U13.28 (36_CS)
- new net APOGEE_SENSE: U13.17 (25_A11_RX6_SDA2)
- new net FLASH_SPI.MISO: U13.14 (12_MISO_MQSL)
- new net FLASH_SPI.MOSI: U13.13 (11_MOSI_CTX1)
- new net FLASH_SPI.SCLK: U13.35 (13_SCK_LED)
- new net FLASH_SPI.nCS: U13.12 (10_CS_MQSR)
- new net GND: BZ1.2 (-), D1.1 (K), D2.1 (K), D3.1 (K), U13.1 (GND), U13.34 (GND), U13.47 (GND)
- new net GPS.EN: U13.11 (9_OUT1C)
- new net GPS.RX: U13.10 (8_TX2_IN1)
- new net GPS.TX: U13.9 (7_RX2_OUT1A)
- new net I2C_SCL: R1.2, U13.41 (19_A5_SCL)
- new net I2C_SDA: R2.2, U13.40 (18_A4_SDA)
- new net LED0: R3.1, U13.4 (2_OUT2)
- new net LED1: R4.1, U13.5 (3_LRCLK2)
- new net LED2: R5.1, U13.6 (4_BCLK2)
- new net MAIN_FIRE: U13.29 (37_CS)
- new net MAIN_SENSE: U13.16 (24_A10_TX6_SCL2)
- new net RADIO.CS: U13.2 (0_RX1_CRX2_CS1)
- new net RADIO.EN: U13.21 (29_TX7)
- new net RADIO.G0: U13.39 (17_A3_TX4_SDA1)
- new net RADIO.G1: U13.38 (16_A2_RX4_SCL1)
- new net RADIO.G2: U13.37 (15_A1_RX3_SPDIF_IN)
- new net RADIO.G3: U13.36 (14_A0_TX3_SPDIF_OUT)
- new net RADIO.G4: U13.33 (41_A17)
- new net RADIO.G5: U13.32 (40_A16)
- new net RADIO.MISO: U13.3 (1_TX1_CTX2_MISO1)
- new net RADIO.MOSI: U13.18 (26_A12_MOSI1)
- new net RADIO.RST: U13.20 (28_RX7)
- new net RADIO.SCK: U13.19 (27_A13_SCK1)
- no-connect marks 0 -> 14
Other:
- note added: "Debug LEDs"
