File: phoenix/mcu.kicad_sch (KiCad schematic)
At the start: 10 parts, among them U13 Teensy4.1

Commit message: Final version for LC2026
Parts:
- added J14: Conn_01x04_Pin, Connector_JST:JST_XH_S4B-XH-A_1x04_P2.50mm_Horizontal, symbol Connector:Conn_01x04_Pin
Connections:
- net +5V: now also J14.1 (Pin_1)
- net GND: now also J14.2 (Pin_2)
- net GPIO7: now reaches U13.7 (5_IN2)
- net GPIO7: now also J14.4 (Pin_4)
- net GPIO8: now reaches U13.8 (6_OUT1D)
- net GPIO8: now also J14.3 (Pin_3)
- no-connect marks 14 -> 12
