File: phoenix/phoenix.kicad_pcb (KiCad board)
At the start: 4 copper layers, 95.5 x 126.4 mm, 172 parts, among them J1 Conn_01x04_Pin, J10 Conn_01x04_Pin, J11 Conn_01x02_Pin, J12 Conn_01x04_Pin, J13 Conn_01x02_Pin, J16 Conn_01x04_Pin, J17 Conn_01x04_Pin, J2 Conn_01x02_Pin, J3 Conn_01x22_Socket, J4 Conn_01x22_Socket, J5 Conn_01x04_Pin, J6 Conn_01x02_Pin, J7 Raspberry_Pi_4, J8 Conn_01x04_Pin, J9 Conn_01x02_Pin, U1 LD1117S33TR_SOT223, U10 VN7140ASTR, U11 VN7140ASTR, U12 BMP581, U13 Teensy4.1, U14 Adafruit_RFM9x, U15 AOZ6605PI-1, U2 LIS3MDLTR, U3 BMP280, U4 LSM6DSOXTR, U5 XTSD04G, U6 MCP9808T-E_MS, U7 Adafruit_Ult_GPS, U8 Adafruit_RFM9x, U9 TPS54386PWPR

Commit message: Final version for LC2026
Parts:
- added J14: Conn_01x04_Pin, Connector_JST:JST_XH_S4B-XH-A_1x04_P2.50mm_Horizontal, F.Cu at (72.4, 43.0)
- moved G*** 24.3 mm to (74.0, 66.6)
- moved C27 3.33 mm to (82.0, 140.2)
- turned C30 to 180 degrees
Connections:
- U13 pad 7: unconnected-(U13-5_IN2-Pad7) -> /MCU/GPIO7
- U13 pad 8: unconnected-(U13-6_OUT1D-Pad8) -> /MCU/GPIO8
Routing:
- net /rpi_power/+3V3: track 0.00 -> 94.8 mm
- net /rpi_power/SPI_CE0: track 0.00 -> 59.4 mm
- net /rpi_power/SPI_CE1: track 0.00 -> 52.3 mm
- net /rpi_power/SPI_MISO: track 0.00 -> 35.5 mm
- net /rpi_power/I2C_SDA: track 0.00 -> 29.7 mm
- net /rpi_power/SPI_MOSI: track 0.00 -> 29.6 mm
- net /rpi_power/I2C_SCL: track 0.00 -> 29.5 mm
- net /rpi_power/EXT_IO: track 0.00 -> 27.2 mm
- net +5V: track 115.4 -> 141.6 mm, vias 1 -> 2
- net /rpi_power/SPI_CLK: track 0.00 -> 25.2 mm
- net /rpi_power/UART_TX: track 0.00 -> 25.0 mm
- net /rpi_power/VBAT: track 0.00 -> 25.0 mm
- net /rpi_power/UART_RX: track 0.00 -> 24.4 mm
- net Net-(BZ2--): track 0.00 -> 14.3 mm
- net /MCU/GPIO8: track 0.00 -> 10.2 mm
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- added copper zone on F.Cu, net /rpi_power/+5V1
- added copper zone on In2.Cu, net /rpi_power/+5V1
- added copper zone on F.Cu, net /rpi_power/LX
